Commit message: race car

File: environment/urdf/differentialDriveCar.urdf (robot description, URDF)
Before this commit: robot miniBox, 5 links, 4 joints
Links:
- removed link front_follow_wheel
- removed link front_follow_wheel_pillar
- added link top_link; collision cylinder length=0.3 radius=0.25; visual cylinder length=0.3 radius=0.25
- link base_link: mass 5 -> 60; geometry collision cylinder length=0.01 radius=0.25; visual cylinder length=0.01 radius=0.25
- link left_wheel: geometry collision cylinder length=0.1 radius=0.1; visual cylinder length=0.1 radius=0.1
- link right_wheel: geometry collision cylinder length=0.1 radius=0.1; visual cylinder length=0.1 radius=0.1
Joints:
- removed joint base_to_front_follow_wheel_pillar
- removed joint front_pillar_to_front_follow_wheel
- added joint joint_top: type continuous, parent base_link, child top_link, origin xyz=0 0 0.15 rpy=0 0 0, axis 0 1 0
- joint joint_left_wheel: origin xyz=-0.1 0.30 0 rpy=0 0 0 -> xyz=0 0.115 0.09 rpy=0 0 0
- joint joint_right_wheel: origin xyz=-0.1 -0.30 0 rpy=0 0 0 -> xyz=0 -0.115 0.09 rpy=0 0 0

Commit message: race car

File: environment/urdf/differentialDriveCar.urdf (robot description, URDF)
Before this commit: robot miniBox, 4 links, 3 joints
Links:
- link top_link: mass None -> 0
