Commit message: step duration 0.1 without collision

File: environment/robots/urdf/differentialDriveCar.urdf (robot description, URDF)
Before this commit: robot miniBox, 4 links, 3 joints
Links:
- link top_link: mass 0 -> 60; geometry collision cylinder length=0.8 radius=0.25; visual cylinder length=0.8 radius=0.25
Joints:
- joint joint_top: origin xyz=0 0 0.15 rpy=0 0 0 -> xyz=0 0 0.4 rpy=0 0 0

Commit message: change height

File: environment/robots/urdf/differentialDriveCar.urdf (robot description, URDF)
Before this commit: robot miniBox, 4 links, 3 joints
Links:
- link top_link: geometry collision cylinder length=0.4 radius=0.25; visual cylinder length=0.4 radius=0.25
Joints:
- joint joint_top: origin xyz=0 0 0.4 rpy=0 0 0 -> xyz=0 0 0.2 rpy=0 0 0

Commit message: modify parameters

File: environment/robots/urdf/differentialDriveCar.urdf (robot description, URDF)
Before this commit: robot miniBox, 4 links, 3 joints
Links:
- link top_link: geometry collision cylinder length=1.7 radius=0.25; visual cylinder length=1.7 radius=0.25
Joints:
- joint joint_top: origin xyz=0 0 0.2 rpy=0 0 0 -> xyz=0 0 0.85 rpy=0 0 0
